File: hardware/botw_pcb/botw_pcb.kicad_sch (KiCad schematic)
At the start: 55 parts, among them M1 Motor_DC, M2 Motor_DC, M3 Motor_DC, M4 Motor_DC, M5 Motor_DC, M6 Motor_DC, M7 Motor_DC, M8 Motor_DC, P1 USB_C_Plug_USB2.0, Q1 S8050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

Commit message: Changed to a new part for mag
Parts:
- C1: value 1 uF -> 1u
- C2: value 10 uF -> 10u
- C3: value 0.1 uF -> 0.1u
- C4, C5: value 10uF -> 10u
- L1: value 2.2uH -> 2.2u
- R10, R11, R12, R13, R14, R15, R18, R8, R9: value 2.2k -> 2k2

Commit message: Transistor footprint was wrong, whoops! Also added in hard iron correction
Parts:
- added R21: 0, Resistor_SMD:R_0603_1608Metric, symbol Device:R_Small_US
- Q1, Q2, Q3, Q4, Q5, Q6, Q7, Q8, Q9: symbol Transistor_BJT:S8050 -> custom:S8050
Connections:
- net +BATT: now also R21.2; no longer BT1.1 (+)
- net GND: now also Q1.2 (E), Q2.2 (E), Q3.2 (E), Q4.2 (E), Q5.2 (E), Q6.2 (E), Q7.2 (E), Q8.2 (E), Q9.2 (E); no longer Q1.3 (C), Q2.3 (C), Q3.3 (C), Q4.3 (C), Q5.3 (C), Q6.3 (C), Q7.3 (C), Q8.3 (C), Q9.3 (C)
- net at R8.1: now also Q1.1 (B); no longer Q1.2 (B)
- net at R12.1: now also Q6.1 (B); no longer Q6.2 (B)
- net at Q5.1 (B): now also R18.1; no longer R2.2
- net at R10.1: now also Q3.1 (B); no longer Q3.2 (B)
- net at R9.1: now also Q2.1 (B); no longer Q2.2 (B)
- net at D5.2 (A), M4.2 (-): now also Q4.3 (C); no longer Q4.1 (E)
- net at D4.2 (A), M3.2 (-): now also Q3.3 (C); no longer Q3.1 (E)
- net at D7.2 (A), M6.2 (-): now also Q7.3 (C); no longer Q7.1 (E)
- net at D2.2 (A), M2.2 (-): now also Q2.3 (C); no longer Q2.1 (E)
- net at D1.2 (A), M1.2 (-): now also Q1.3 (C); no longer Q1.1 (E)
- net at R15.1: now also Q9.1 (B); no longer Q9.2 (B)
- net at R13.1: now also Q7.1 (B); no longer Q7.2 (B)
- net at D9.2 (A), M8.2 (-): now also Q9.3 (C); no longer Q9.1 (E)
- net at D8.2 (A), M7.2 (-): now also Q8.3 (C); no longer Q8.1 (E)
- net at R14.1: now also Q8.1 (B); no longer Q8.2 (B)
- net at D6.2 (A), M5.2 (-): now also Q6.3 (C); no longer Q6.1 (E)
- net at R11.1: now also Q4.1 (B); no longer Q4.2 (B)
- new net: Q5.3 (C), R2.2
- new net: BT1.1 (+), R21.1
Other:
- moved on the sheet: C2, C3, C4, C5, D10, L1, R16, R17, R3, R4, SW1, U2
